Commit message: scale the collision sphere into 0.9 times

File: wrs/robot_sim/robots/xarmlite6_wg/xarm6_sphere_visuals.urdf (robot description, URDF)
Before this commit: robot xarm_lite6, 9 links, 8 joints
Links:
- link base_link: geometry collision sphere radius=0.02730395; collision sphere radius=0.0407911
- link link1: geometry collision sphere radius=0.03091205; collision sphere radius=0.0355167
- link link2: geometry collision sphere radius=0.03880085; collision sphere radius=0.0426379
- link link3: geometry collision sphere radius=0.04061155; collision sphere radius=0.0460351
- link link4: geometry collision sphere radius=0.0302689; collision sphere radius=0.03474245
- link link5: geometry collision sphere radius=0.03354545; collision sphere radius=0.03450685
- link link6: geometry collision sphere radius=0.0180519; collision sphere radius=0.0221141
- link spine_miller: geometry collision sphere radius=0.01492735; collision sphere radius=0.0185906

Commit message: scale the collision sphere into 0.9 times

File: wrs/robot_sim/robots/xarmlite6_wg/xarm6_sphere_visuals.urdf (robot description, URDF)
Before this commit: robot xarm_lite6, 9 links, 8 joints
Links:
- link spine_miller: geometry collision sphere radius=0.01492735; collision sphere radius=0.0361228

Commit message: now can detect the collison, but the code seems redundant

File: wrs/robot_sim/robots/xarmlite6_wg/xarm6_sphere_visuals.urdf (robot description, URDF)
Before this commit: robot xarm_lite6, 9 links, 8 joints
Links:
- link link6: geometry visual mesh filename=package://xarm_lite6_description/meshes/link6.stl
- link spine_miller: geometry collision sphere radius=0.01492735; collision sphere radius=0.033225
