Commit message: fixing foam axis

File: wrs/robot_sim/robots/franka_research_3/franka_research_3_sphere_visuals.urdf (robot description, URDF)
Before this commit: robot franka_research_3, 8 links, 7 joints
Links:
- link link3: geometry visual mesh filename=/home/lqin/wrs_xinyi/wrs/robot_sim/manipulators/franka_rese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
- link link4: geometry visual mesh filename=/home/lqin/wrs_xinyi/wrs/robot_sim/manipulators/franka_rese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
- link link5: geometry visual mesh filename=/home/lqin/wrs_xinyi/wrs/robot_sim/manipulators/franka_rese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
- link link6: geometry visual mesh filename=/home/lqin/wrs_xinyi/wrs/robot_sim/manipulators/franka_rese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
- link link7: geometry visual mesh filename=/home/lqin/wrs_xinyi/wrs/robot_sim/manipulators/franka_rese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
Joints:
- joint joint1: origin xyz=0 0 0.333 rpy=0 0 0 -> xyz=0 0 0.133 rpy=0 0 0
- joint joint2: origin xyz=0 0 0 rpy=-1.57079632679 0 0 -> xyz=0 0 0.2 rpy=-1.57079632679 0 0

Commit message: [franka foam ckpt] hand revised all the parameters

File: wrs/robot_sim/robots/franka_research_3/franka_research_3_sphere_visuals.urdf (robot description, URDF)
Before this commit: robot franka_research_3, 8 links, 7 joints
Links:
- link link3: geometry collision sphere radius=0.054807; collision sphere radius=0.057881
- link link4: geometry collision sphere radius=0.054192; collision sphere radius=0.061485
- link link5: geometry collision sphere radius=0.045514; collision sphere radius=0.047317
- link link6: geometry collision sphere radius=0.044327; collision sphere radius=0.053238
- link link7: geometry collision sphere radius=0.029962; collision sphere radius=0.030309
Joints:
- joint joint1: origin xyz=0 0 0.133 rpy=0 0 0 -> xyz=0 0 0.135 rpy=0 0 0
- joint joint3: origin xyz=0 -0.316 0 rpy=1.57079632679 0 0 -> xyz=0 -0.2 0 rpy=1.57079632679 0 0
- joint joint4: origin xyz=0.0825 0 0 rpy=1.57079632679 0 0 -> xyz=0.0825 0 0.12 rpy=1.57079632679 0 0
- joint joint5: origin xyz=-0.0825 0.384 0 rpy=-1.57079632679 0 0 -> xyz=-0.0825 0.12 0 rpy=-1.57079632679 0 0
- joint joint6: origin xyz=0 0 0 rpy=1.57079632679 0 0 -> xyz=0 0.012 0.253 rpy=1.57079632679 0 0
- joint joint7: origin xyz=0.088 0 0 rpy=1.57079632679 0 0 -> xyz=0.088 -0.055 0 rpy=1.57079632679 0 0

Commit message: franka hand calibrated

File: wrs/robot_sim/robots/franka_research_3/franka_research_3_sphere_visuals.urdf (robot description, URDF)
Before this commit: robot franka_research_3, 9 links, 8 joints
Links:
- added link left_finger; collision sphere radius=0.009618; collision sphere radius=0.009655
- added link right_finger; collision sphere radius=0.009618; collision sphere radius=0.009655
- link hand: geometry collision sphere radius=0.039441; collision sphere radius=0.039817
Joints:
- added joint finger_joint1: type prismatic, parent hand, child left_finger, origin xyz=-0.011 0.005 0.115 rpy=0 0 0, axis 0 1 0, limit lower=0.0 upper=0.04 effort=50 velocity=0.2
- added joint finger_joint2: type prismatic, parent hand, child right_finger, origin xyz=0 0.011 0.115 rpy=0 0 3.14159265359, axis 0 1 0, limit lower=0.0 upper=0.04 effort=50 velocity=0.2
- joint franka_fixed_joint: origin xyz=0 0 0.058 rpy=0 0 0.5 -> xyz=0 0 0 rpy=0 0 0

Commit message: individual test passed

File: wrs/robot_sim/robots/franka_research_3/franka_research_3_sphere_visuals.urdf (robot description, URDF)
Before this commit: robot franka_research_3, 11 links, 10 joints
Joints:
- joint finger_joint1: origin xyz=-0.011 0.005 0.115 rpy=0 0 0 -> xyz=0 0.01 0.055 rpy=0 0 0
- joint finger_joint2: origin xyz=0 0.011 0.115 rpy=0 0 3.14159265359 -> xyz=0 0.01 0.055 rpy=0 0 3.14159265359
- joint franka_fixed_joint: origin xyz=0 0 0 rpy=0 0 0 -> xyz=0 0 0.058 rpy=0 0 0.5

Commit message: ok for id check, not ok for whole

File: wrs/robot_sim/robots/franka_research_3/franka_research_3_sphere_visuals.urdf (robot description, URDF)
Before this commit: robot franka_research_3, 11 links, 10 joints
Links:
- link left_finger: geometry collision sphere radius=0.001132; collision sphere radius=0.002618
- link link5: geometry collision sphere radius=0.045514; collision sphere radius=0.047317
- link right_finger: geometry collision sphere radius=0.008966; collision sphere radius=0.009618
Joints:
- joint finger_joint1: origin xyz=0 0.01 0.055 rpy=0 0 0 -> xyz=0 0.01 0.06 rpy=0 0 0
- joint finger_joint2: origin xyz=0 0.01 0.055 rpy=0 0 3.14159265359 -> xyz=0 0.01 0.06 rpy=0 0 3.14159265359

Commit message: [franka ckpt cc check gpu] finished all calibrations, delete the fingers bcs its so annoying

File: wrs/robot_sim/robots/franka_research_3/franka_research_3_sphere_visuals.urdf (robot description, URDF)
Before this commit: robot franka_research_3, 11 links, 10 joints
Links:
- link left_finger: geometry visual mesh filename=/home/lqin/wrs_xinyi/wrs/robot_sim/end_effectors/grippers/f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
- link right_finger: geometry visual mesh filename=/home/lqin/wrs_xinyi/wrs/robot_sim/end_effectors/grippers/f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
Joints:
- joint finger_joint1: origin xyz=0 0.01 0.06 rpy=0 0 0 -> xyz=0 0.035 0.06 rpy=0 0 0
- joint finger_joint2: origin xyz=0 0.01 0.06 rpy=0 0 3.14159265359 -> xyz=0 0.035 0.06 rpy=0 0 3.14159265359
- joint franka_fixed_joint: origin xyz=0 0 0.058 rpy=0 0 0.5 -> xyz=0.025 0.01 0.058 rpy=0 0 0.5
