Commit message: fr3 cali didnt finished, jnt 8

File: wrs/robot_sim/robots/franka_research_3/franka_research_3_ccsphere.urdf (robot description, URDF)
Before this commit: robot franka_research_3, 11 links, 10 joints
Links:
- link link5: geometry collision sphere radius=0.045514; collision sphere radius=0.047317
- link link6: geometry collision sphere radius=0.039894; collision sphere radius=0.047914
Joints:
- joint franka_fixed_joint: origin xyz=0.025 0.01 0.058 rpy=0 0 0.5 -> xyz=0.025 0.03 0.058 rpy=0 0 0.78539816339
- joint joint7: origin xyz=0.088 -0.045 0 rpy=1.57079632679 0.5 0 -> xyz=0.088 -0.045 0 rpy=1.57079632679 0.78539816339 0

Commit message: start debugging fr3 urdf

File: wrs/robot_sim/robots/franka_research_3/franka_research_3_ccsphere.urdf (robot description, URDF)
Before this commit: robot franka_research_3, 11 links, 10 joints
Links:
- link left_finger: geometry collision sphere radius=0.001132; collision sphere radius=0.002618
Joints:
- joint finger_joint1: origin xyz=0 0.035 0.06 rpy=0 0 0 -> xyz=0 0.01 0.0584 rpy=0 0 0
- joint franka_fixed_joint: axis (none) -> 0 1 0; origin xyz=0.025 0.03 0.058 rpy=0 0 0.78539816339 -> xyz=0 0 0.0584 rpy=0 0 0.78539816339

Commit message: all accurate but link6

File: wrs/robot_sim/robots/franka_research_3/franka_research_3_ccsphere.urdf (robot description, URDF)
Before this commit: robot franka_research_3, 11 links, 10 joints
Links:
- link right_finger: geometry collision sphere radius=0.008966; collision sphere radius=0.009618
Joints:
- joint finger_joint1: limit lower=0.0 upper=0.04 effort=50 velocity=0.2 -> lower=0.0 upper=0.015 effort=50 velocity=0.2; origin xyz=0 0.01 0.0584 rpy=0 0 0 -> xyz=0 0 0.0584 rpy=0 0 0
- joint finger_joint2: limit lower=0.0 upper=0.04 effort=50 velocity=0.2 -> lower=0.0 upper=0.015 effort=50 velocity=0.2; origin xyz=0 0.035 0.06 rpy=0 0 3.14159265359 -> xyz=0 0 0 rpy=0 0 3.14159265359
- joint franka_fixed_joint: origin xyz=0 0 0.0584 rpy=0 0 0.78539816339 -> xyz=0 0 0.107 rpy=0 0 0
- joint joint1: origin xyz=0 0 0.135 rpy=0 0 0 -> xyz=0 0 0.333 rpy=0 0 0
- joint joint2: origin xyz=0 0 0.2 rpy=-1.57079632679 0 0 -> xyz=0 0 0 rpy=-1.57079632679 0 0
- joint joint3: origin xyz=0 -0.2 0 rpy=1.57079632679 0 0 -> xyz=0 -0.316 0 rpy=1.57079632679 0 0
- joint joint4: origin xyz=0.0825 0 0.12 rpy=1.57079632679 0 0 -> xyz=0.0825 0 0 rpy=1.57079632679 0 0
- joint joint5: origin xyz=-0.0825 0.12 0 rpy=-1.57079632679 0 0 -> xyz=-0.0825 0.384 0 rpy=-1.57079632679 0 0
- joint joint6: origin xyz=0 0.012 0.253 rpy=1.57079632679 0 0 -> xyz=0 0 0 rpy=1.57079632679 0 0
- joint joint7: origin xyz=0.088 -0.045 0 rpy=1.57079632679 0.78539816339 0 -> xyz=0.088 0 0 rpy=1.57079632679 0 0

Commit message: [cccckkkkppppttt] fr3 cc checker finally finished

File: wrs/robot_sim/robots/franka_research_3/franka_research_3_ccsphere.urdf (robot description, URDF)
Before this commit: robot franka_research_3, 11 links, 10 joints
Links:
- link right_finger: geometry collision sphere radius=0.001132; collision sphere radius=0.002618
Joints:
- joint finger_joint2: origin xyz=0 0 0 rpy=0 0 3.14159265359 -> xyz=0 0 0.0584 rpy=0 0 3.14159265359
